Commit message: Xacro to sdf

File: world/xacro/maze_world.xacro (robot description, xacro)
@@ -1,4 +1,7 @@
 <?xml version="1.0"?>
-<sdf version="1.10">
+<xacro:sdf version="1.10"
+  xmlns:xacro="http://ros.org/wiki/xacro">
+  <xacro:include filename="$(find minor)/world/xacro/start_goal.xacro" />
+  <xacro:include filename="$(find minor)/world/xacro/wall.xacro" />
   <world name="maze_world">
     <!-- Physics & plugins -->
@@ -51,96 +54,8 @@
     <!-- === Maze walls === -->
     <!-- Outer boundary -->
-    <model name="wall_bottom">
-      <static>true</static>
-      <pose>0 -5 0 0 0 1.5708</pose>
-      <link name="link">
-        <visual name="visual">
-          <geometry>
-            <box>
-              <size>0.5 10.0 4.0</size>
-            </box>
-          </geometry>
-          <material>
-            <ambient>0 0 1 1</ambient>
-          </material>
-        </visual>
-        <collision name="collision">
-          <geometry>
-            <box>
-              <size>0.5 10.0 4.0</size>
-            </box>
-          </geometry>
-        </collision>
-      </link>
-    </model>
-    <model name="wall_top">
-      <static>true</static>
-      <pose>0 5 0 0 0 1.5708</pose>
-      <link name="link">
-        <visual name="visual">
-          <geometry>
-            <box>
-              <size>0.5 10.0 4.0</size>
-            </box>
-          </geometry>
-          <material>
-            <ambient>0 0 1 1</ambient>
-          </material>
-        </visual>
-        <collision name="collision">
-          <geometry>
-            <box>
-              <size>0.5 10.0 4.0</size>
-            </box>
-          </geometry>
-        </collision>
-      </link>
-    </model>
-    <model name="wall_left">
-      <static>true</static>
-      <pose>-5 0 0 0 0 0</pose>
-      <link name="link">
-        <visual name="visual">
-          <geometry>
-            <box>
-              <size>0.5 10.0 4.0</size>
-            </box>
-          </geometry>
-          <material>
-            <ambient>0 0 1 1</ambient>
-          </material>
-        </visual>
-        <collision name="collision">
-          <geometry>
-            <box>
-              <size>0.5 10.0 4.0</size>
-            </box>
-          </geometry>
-        </collision>
-      </link>
-    </model>
-    <model name="wall_right">
-      <static>true</static>
-      <pose>5 0 0 0 0 0</pose>
-      <link name="link">
-        <visual name="visual">
-          <geometry>
-            <box>
-              <size>0.5 10.0 4.0</size>
-            </box>
-          </geometry>
-          <material>
-            <ambient>0 0 1 1</ambient>
-          </material>
-        </visual>
-        <collision name="collision">
-          <geometry>
-            <box>
-              <size>0.5 10.0 4.0</size>
-            </box>
-          </geometry>
-        </collision>
-      </link>
-    </model>
+    <xacro:wall name="wall_bottom"
+      pose="0 -5 0 0 0 1.5708"
+      size="0.5 10.0 4.0"
+      color="0 0 1 1" />
     <!-- Origin Marker -->
     <model name="Origin">
@@ -162,72 +77,6 @@
     </model>
     <!-- === Start & Goal markers === -->
-    <model name="Start">
-      <static>true</static>
-      <pose>-4 -4 2 0 0 0</pose>
-      <link name="link">
-        <!-- Sphere part (head of the pin) -->
-        <visual name="pin_head">
-          <pose>0 0 0.4 0 0 0</pose>
-          <geometry>
-            <sphere>
-              <radius>0.3</radius>
-            </sphere>
-          </geometry>
-          <material>
-            <ambient>0 0 1 1</ambient>
-            <diffuse>0 0 1 1</diffuse>
-          </material>
-        </visual>
-        <!-- Cone part (tip of the pin) -->
-        <visual name="pin_tip">
-          <pose>0 0 -0.2 0 0 0</pose>
-          <geometry>
-            <mesh>
-              <uri>stl/cone.stl</uri>
-              <!-- optional: adjust mesh scaling if you want a larger/smaller cone -->
-              <!-- <scale>1 1 1</scale> -->
-            </mesh>
-          </geometry>
-          <material>
-            <ambient>0 0 1 1</ambient>
-            <diffuse>0 0 1 1</diffuse>
-          </material>
-        </visual>
-      </link>
-    </model>
-    <model name="Goal">
-      <static>true</static>
-      <pose>-4 4 2 0 0 0</pose>
-      <link name="link">
-        <!-- Sphere part (head of the pin) -->
-        <visual name="pin_head">
-          <pose>0 0 0.4 0 0 0</pose>
-          <geometry>
-            <sphere>
-              <radius>0.3</radius>
-            </sphere>
-          </geometry>
-          <material>
-            <ambient>0 1 0 1</ambient>
-            <diffuse>0 1 0 1</diffuse>
-          </material>
-        </visual>
-        <!-- Cone part (tip of the pin) -->
-        <visual name="pin_tip">
-          <pose>0 0 -0.2 0 0 0</pose>
-          <geometry>
-            <mesh>
-              <uri>stl/cone.stl</uri>
-              <!-- optional: adjust mesh scaling if you want a larger/smaller cone -->
-              <!-- <scale>1 1 1</scale> -->
-            </mesh>
-          </geometry>
-          <material>
-            <ambient>0 1 0 1</ambient>
-            <diffuse>0 1 0 1</diffuse>
-          </material>
-        </visual>
-      </link>
-    </model>
+    <xacro:location_pin name="Start" pose="-4 -4 2 0 0 0" color="0 0 1 1" />
+    <xacro:location_pin name="Goal" pose="-4  4 2 0 0 0" color="0 1 0 1" />
     <!-- Vehicle Model -->
     <model name='vehicle_blue' canonical_link='chassis'>
@@ -462,3 +311,3 @@
     </model>
   </world>
-</sdf>
+</xacro:sdf>

Commit message: Xacro to SDF - Maze env update

File: world/xacro/maze_world.xacro (robot description, xacro)
@@ -55,31 +55,21 @@
     <!-- Outer boundary -->
     <xacro:wall name="wall_bottom"
-      pose="0 -5 0 0 0 1.5708"
-      size="0.5 10.0 4.0"
-      color="0 0 1 1" />
-    <!-- Origin Marker -->
-    <model name="Origin">
-      <static>true</static>
-      <pose>0 0 0 0 0 0</pose>
-      <link name="link">
-        <visual name="sphere">
-          <geometry>
-            <sphere>
-              <radius>0.3</radius>
-            </sphere>
-          </geometry>
-          <material>
-            <ambient>1 0 0 1</ambient>
-            <diffuse>1 0 0 1</diffuse>
-          </material>
-        </visual>
-      </link>
-    </model>
+      pose="0 -7 0 0 0 1.5708"
+      length="14.0" />
+    <xacro:wall name="wall_left"
+      pose="-7 0 0 0 0 0"
+      length="14.5" />
+    <xacro:wall name="wall_right"
+      pose="7 0 0 0 0 0"
+      length="14.5" />
+    <xacro:wall name="wall_top"
+      pose="0 7 0 0 0 1.5708"
+      length="14.0" />
     <!-- === Start & Goal markers === -->
-    <xacro:location_pin name="Start" pose="-4 -4 2 0 0 0" color="0 0 1 1" />
-    <xacro:location_pin name="Goal" pose="-4  4 2 0 0 0" color="0 1 0 1" />
+    <xacro:location_pin name="Start" pose="-5 -5 2 0 0 0" color="0 0 1 1" />
+    <xacro:location_pin name="Goal" pose="-5 5 2 0 0 0" color="0 1 0 1" />
     <!-- Vehicle Model -->
     <model name='vehicle_blue' canonical_link='chassis'>
-      <pose relative_to='world'>-4 -4 0 0 0 0</pose>
+      <pose relative_to='world'>-5 -5 0 0 0 0</pose>
       <link name='chassis'>
         <pose relative_to='__model__'>0.5 0 0.4 0 0 0</pose>

File: world/xacro/wall.xacro (robot description, xacro)
@@ -1,6 +1,10 @@
 <?xml version="1.0"?>
 <xacro:sdf version="1.10" xmlns:xacro="http://ros.org/wiki/xacro">
-  <!-- Macro for a wall -->
-  <xacro:macro name="wall" params="name pose size color">
+  <!-- ===== Global wall properties ===== -->
+  <xacro:property name="wall_height" value="4.0"/>
+  <xacro:property name="wall_thickness" value="0.5"/>
+  <xacro:property name="wall_color" value="0 0 1 1"/>
+  <!-- ===== Macro for a wall ===== -->
+  <xacro:macro name="wall" params="name pose length">
     <model name="${name}">
       <static>true</static>
@@ -11,10 +15,10 @@
           <geometry>
             <box>
-              <size>${size}</size>
+              <size>${wall_thickness} ${length} ${wall_height}</size>
             </box>
           </geometry>
           <material>
-            <ambient>${color}</ambient>
-            <diffuse>${color}</diffuse>
+            <ambient>${wall_color}</ambient>
+            <diffuse>${wall_color}</diffuse>
             <specular>0.2 0.2 0.2 1</specular>
           </material>
@@ -24,5 +28,5 @@
           <geometry>
             <box>
-              <size>${size}</size>
+              <size>${wall_thickness} ${length} ${wall_height}</size>
             </box>
           </geometry>

Commit message: Maze world Updated

File: world/xacro/maze_world.xacro (robot description, xacro)
@@ -16,5 +16,5 @@
     </plugin>
     <!-- Custom GUI for Video Recording -->
-    <gui fullscreen="1">
+    <gui fullscreen="0">
       <!-- 3D scene -->
       <plugin filename="MinimalScene" name="3D View">
@@ -262,4 +262,7 @@
       pose="0.5 0.5 0 0 0 1.5708"
       length="7.0" />
+    <xacro:wall name="wall_4"
+      pose="0.75 -1.125 2 0 1.5708 0"
+      length="12.25" wall_height="16" />
     <!-- === Start & Goal markers === -->
     <xacro:location_pin name="Start" pose="-11 -5 2 0 0 0" color="1 0 0 1" />

File: world/xacro/wall.xacro (robot description, xacro)
@@ -2,9 +2,9 @@
 <xacro:sdf version="1.10" xmlns:xacro="http://ros.org/wiki/xacro">
   <!-- ===== Global wall properties ===== -->
-  <xacro:property name="wall_height" value="4.0"/>
-  <xacro:property name="wall_thickness" value="0.5"/>
-  <xacro:property name="wall_color" value="0 0 1 1"/>
+  <!-- <xacro:property name="wall_height" value="4.0" /> -->
+  <xacro:property name="wall_thickness" value="0.5" />
+  <xacro:property name="wall_color" value="0 0 1 1" />
   <!-- ===== Macro for a wall ===== -->
-  <xacro:macro name="wall" params="name pose length">
+  <xacro:macro name="wall" params="name pose length wall_height:=4.0">
     <model name="${name}">
       <static>true</static>
